File: pcb/wfkbd.kicad_pcb (KiCad board)
At the start: 2 copper layers, 114 parts, among them J1 MJ-4PP-9, P1 LED, SW1 KEY, SW10 KEY, SW11 KEY, SW12 KEY, SW13 KEY, SW14 KEY, SW15 KEY, SW16 KEY, SW17 KEY, SW18 KEY, SW19 KEY, SW2 KEY, SW20 KEY, SW21 KEY, SW22 KEY, SW23 KEY, SW24 KEY, SW25 KEY, SW26 KEY, SW27 KEY, SW28 KEY, SW29 KEY, SW3 KEY, SW30 KEY, SW31 KEY, SW32 KEY, SW33 KEY, SW34 KEY, SW35 KEY, SW4 KEY, SW5 KEY, SW6 KEY, SW7 KEY, SW8 KEY, SW9 KEY, U1 ProMicro

Commit message: Add pcbnew files
Parts:
- removed CJ1, CJ15, CJ22, CJ8: col0, kbd:1pin_conn
- removed CJ10, CJ17, CJ24, CJ3: col2, kbd:1pin_conn
- removed CJ11, CJ18, CJ25, CJ4: col3, kbd:1pin_conn
- removed CJ12, CJ19, CJ26, CJ5: col4, kbd:1pin_conn
- removed CJ13, CJ20, CJ27, CJ6: col5, kbd:1pin_conn
- removed CJ14, CJ21, CJ28, CJ7: col6, kbd:1pin_conn
- removed CJ16, CJ2, CJ23, CJ9: col1, kbd:1pin_conn
- removed P1: LED, kbd:StripLED_rev
- removed RJ1, RJ10, RJ2, RJ3, RJ4, RJ5, RJ6, RJ7, RJ8, RJ9: row0, kbd:1pin_conn
- added C1: VCC, kbd:1pin_conn, F.Cu at (88.5, 42.0)
- added C2: GND, kbd:1pin_conn, F.Cu at (91.0, 42.0)
- added C3: LED, kbd:1pin_conn, F.Cu at (93.5, 42.0)
- moved D1 119.9 mm to (42.0, 50.0), turned to 270 degrees
- moved SW1 112.8 mm to (50.0, 50.0), turned to 180 degrees
- moved D8 112.4 mm to (42.0, 69.0), turned to 270 degrees
- moved D29 108.6 mm to (42.0, 126.0), turned to 270 degrees
- moved D15 107.8 mm to (42.0, 88.0), turned to 270 degrees
- moved D22 106.5 mm to (42.0, 107.0), turned to 270 degrees
- moved SW8 104.9 mm to (50.0, 69.0), turned to 180 degrees
- moved SW29 100.7 mm to (50.0, 126.0), turned to 180 degrees
- moved SW15 100.0 mm to (50.0, 88.0), turned to 180 degrees
- moved SW22 98.5 mm to (50.0, 107.0), turned to 180 degrees
- moved SW2 96.7 mm to (69.0, 50.0), turned to 180 degrees
- moved D2 90.2 mm to (77.0, 50.0), turned to 270 degrees
- moved D3 87.9 mm to (80.0, 50.0), turned to 270 degrees
- moved SW9 87.3 mm to (69.0, 69.0), turned to 180 degrees
- moved SW30 82.2 mm to (69.0, 126.0), turned to 180 degrees
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Routing:
- net row4: track 0.00 -> 276.4 mm, vias 0 -> 8
- net col0: track 0.00 -> 262.2 mm
- net row3: track 0.00 -> 254.8 mm, vias 0 -> 4
- net col6: track 0.00 -> 216.0 mm, vias 0 -> 4
- net row2: track 0.00 -> 210.4 mm, vias 0 -> 2
- net row1: track 0.00 -> 207.2 mm
- net row0: track 0.00 -> 203.8 mm
- net col1: track 0.00 -> 200.4 mm, vias 0 -> 4
- net col5: track 0.00 -> 182.4 mm, vias 0 -> 2
- net col2: track 0.00 -> 180.9 mm, vias 0 -> 2
- net col4: track 0.00 -> 164.1 mm
- net col3: track 0.00 -> 159.4 mm
- net VCC: track 0.00 -> 73.7 mm
- net GND: track 0.00 -> 57.6 mm
- net data: track 0.00 -> 46.6 mm, vias 0 -> 2
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Other:
- board outline added: 132 x 98 mm

Commit message: To simply
Parts:
- RSW1: footprint kbd:SW_3.5x6.0_TH -> Keebio-Parts:SW_Tactile_SPST_Angled_MJTP1117
- moved RSW1 2.50 mm to (118.0, 39.2)
Routing:
- net reset: track 14.1 -> 8.13 mm
- net GND: track 57.6 -> 60.1 mm
- net row0: track 203.8 -> 206.2 mm
- net VCC: track 73.7 -> 74.4 mm
- net data: track 46.6 -> 47.2 mm

Commit message: Add holes
Parts:
- added ?: , kbd:LegoHole, F.Cu at (59.5, 59.5)
- added ?: , kbd:LegoHole, F.Cu at (154.5, 59.5)
- added ?: , kbd:LegoHole, F.Cu at (154.5, 78.5)
- added ?: , kbd:LegoHole, F.Cu at (135.5, 78.5)
- added ?: , kbd:LegoHole, F.Cu at (135.5, 97.5)
- added ?: , kbd:LegoHole, F.Cu at (154.5, 97.5)
- added ?: , kbd:LegoHole, F.Cu at (154.5, 116.5)
- added ?: , kbd:LegoHole, F.Cu at (135.5, 116.5)
- added ?: , kbd:LegoHole, F.Cu at (78.5, 59.5)
- added ?: , kbd:LegoHole, F.Cu at (59.5, 116.5)
- added ?: , kbd:LegoHole, F.Cu at (78.5, 116.5)
- added ?: , kbd:LegoHole, F.Cu at (78.5, 97.5)
- added ?: , kbd:LegoHole, F.Cu at (59.5, 97.5)
- added ?: , kbd:LegoHole, F.Cu at (59.5, 78.5)
- added ?: , kbd:LegoHole, F.Cu at (78.5, 78.5)
- added ?: , kbd:LegoHole, F.Cu at (135.5, 59.5)

Commit message: To all green DRC
Routing:
- net col0: track 262.2 -> 264.7 mm
- net row1: track 207.2 -> 205.0 mm
- net data: track 47.2 -> 49.3 mm
- net row3: track 254.8 -> 256.8 mm
- net col1: track 200.4 -> 201.7 mm
- net col6: track 216.0 -> 217.0 mm
- net row0: track 206.2 -> 205.3 mm
- net col5: track 182.4 -> 183.2 mm
Changed lines of the file:
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@@
   (general
     (links 578)
-    (no_connects 4)
-    (area 40.924999 36.924999 173.075001 135.075001)
+    (no_connects 3)
+    (area 39.275 35.149999 174.2625 135.275001)
     (thickness 1.6)
     (drawings 336)
-    (tracks 1293)
+    (tracks 1322)
     (zones 0)
     (modules 94)
@@
   (segment (start 63.75 43.5) (end 82.75 43.5) (width 0.25) (layer B.Cu) (net 1))
   (segment (start 61 46.25) (end 63.75 43.5) (width 0.25) (layer B.Cu) (net 1))
-  (segment (start 61 87.5) (end 61 46.25) (width 0.25) (layer B.Cu) (net 1))
+  (segment (start 61 87.5) (end 61 81.5) (width 0.25) (layer B.Cu) (net 1))
+  (segment (start 61 81.5) (end 62.5 80) (width 0.25) (layer B.Cu) (net 1))
+  (segment (start 62.5 80) (end 62.5 77) (width 0.25) (layer B.Cu) (net 1))
+  (segment (start 62.5 77) (end 61 75.5) (width 0.25) (layer B.Cu) (net 1))
+  (segment (start 61 75.5) (end 61 62.5) (width 0.25) (layer B.Cu) (net 1))
+  (segment (start 61 62.5) (end 62.5 61) (width 0.25) (layer B.Cu) (net 1))
+  (segment (start 62.5 61) (end 62.5 58) (width 0.25) (layer B.Cu) (net 1))
+  (segment (start 62.5 58) (end 61 56.5) (width 0.25) (layer B.Cu) (net 1))
+  (segment (start 61 56.5) (end 61 46.25) (width 0.25) (layer B.Cu) (net 1))
   (segment (start 60.5 88) (end 61 87.5) (width 0.25) (layer B.Cu) (net 1))
   (segment (start 58.5 88) (end 60.5 88) (width 0.25) (layer B.Cu) (net 1))
@@
   (via (at 110.25 57.5) (size 0.6) (drill 0.4) (layers F.Cu B.Cu) (net 2))
   (segment (start 110.25 57.5) (end 108.75 57.5) (width 0.25) (layer F.Cu) (net 2))
-  (segment (start 87.25 61.5) (end 71.54 61.5) (width 0.25) (layer B.Cu) (net 2))
+  (segment (start 87.25 61.5) (end 81.5 61.5) (width 0.25) (layer B.Cu) (net 2))
+  (segment (start 81.5 61.5) (end 80 63) (width 0.25) (layer B.Cu) (net 2))
+  (segment (start 80 63) (end 77 63) (width 0.25) (layer B.Cu) (net 2))
+  (segment (start 77 63) (end 75.5 61.5) (width 0.25) (layer B.Cu) (net 2))
+  (segment (start 75.5 61.5) (end 71.54 61.5) (width 0.25) (layer B.Cu) (net 2))
   (via (at 87.25 61.5) (size 0.6) (drill 0.4) (layers F.Cu B.Cu) (net 2))
   (segment (start 88.75 61.5) (end 87.25 61.5) (width 0.25) (layer F.Cu) (net 2))
@@
   (segment (start 129.81 128.61) (end 129.81 128.54) (width 0.25) (layer B.Cu) (net 5))
   (segment (start 114.62 62.19) (end 125.19 62.19) (width 0.25) (layer B.Cu) (net 6))
-  (segment (start 126.75 62.25) (end 145 62.25) (width 0.25) (layer B.Cu) (net 6))
+  (segment (start 126.75 62.25) (end 132.5 62.25) (width 0.25) (layer B.Cu) (net 6))
+  (segment (start 132.5 62.25) (end 133.5 63.25) (width 0.25) (layer B.Cu) (net 6))
+  (segment (start 133.5 63.25) (end 137.5 63.25) (width 0.25) (layer B.Cu) (net 6))
+  (segment (start 137.5 63.25) (end 138.5 62.25) (width 0.25) (layer B.Cu) (net 6))
+  (segment (start 138.5 62.25) (end 145 62.25) (width 0.25) (layer B.Cu) (net 6))
   (via (at 126.75 62.25) (size 0.6) (drill 0.4) (layers F.Cu B.Cu) (net 6))
   (segment (start 125.25 62.25) (end 126.75 62.25) (width 0.25) (layer F.Cu) (net 6))
@@
   (segment (start 129.25 80.5) (end 127.75 80.5) (width 0.25) (layer F.Cu) (net 7))
   (via (at 129.25 80.5) (size 0.6) (drill 0.4) (layers F.Cu B.Cu) (net 7))
-  (segment (start 146.75 80.5) (end 129.25 80.5) (width 0.25) (layer B.Cu) (net 7))
+  (segment (start 146.75 80.5) (end 138.5 80.5) (width 0.25) (layer B.Cu) (net 7))
+  (segment (start 138.5 80.5) (end 137.25 81.75) (width 0.25) (layer B.Cu) (net 7))
+  (segment (start 137.25 81.75) (end 133.75 81.75) (width 0.25) (layer B.Cu) (net 7))
+  (segment (start 133.75 81.75) (end 132.5 80.5) (width 0.25) (layer B.Cu) (net 7))
+  (segment (start 132.5 80.5) (end 129.25 80.5) (width 0.25) (layer B.Cu) (net 7))
   (via (at 146.75 80.5) (size 0.6) (drill 0.4) (layers F.Cu B.Cu) (net 7))
   (segment (start 148.25 80.5) (end 146.75 80.5) (width 0.25) (layer F.Cu) (net 7))
@@
   (segment (start 171.94 46.19) (end 169.25 43.5) (width 0.25) (layer F.Cu) (net 8))
   (segment (start 142.69 61) (end 141.19 59.5) (width 0.25) (layer F.Cu) (net 8))
-  (segment (start 152 61) (end 142.69 61) (width 0.25) (layer F.Cu) (net 8))
-  (segment (start 152.5 60.5) (end 152 61) (width 0.25) (layer F.Cu) (net 8))
-  (segment (start 152.5 51) (end 152.5 60.5) (width 0.25) (layer F.Cu) (net 8))
-  (segment (start 153.5 50) (end 152.5 51) (width 0.25) (layer F.Cu) (net 8))
+  (segment (start 150.5 61) (end 142.69 61) (width 0.25) (layer F.Cu) (net 8))
+  (segment (start 151.5 60) (end 150.5 61) (width 0.25) (layer F.Cu) (net 8))
+  (segment (start 151.5 52) (end 151.5 60) (width 0.25) (layer F.Cu) (net 8))
+  (segment (start 153.5 50) (end 151.5 52) (width 0.25) (layer F.Cu) (net 8))
   (segment (start 155.5 50) (end 153.5 50) (width 0.25) (layer F.Cu) (net 8))
   (segment (start 156 49.5) (end 155.5 50) (width 0.25) (layer F.Cu) (net 8))
@@
   (segment (start 96 58) (end 85.69 58) (width 0.25) (layer F.Cu) (net 8))
   (segment (start 99.43 54.57) (end 96 58) (width 0.25) (layer F.Cu) (net 8) (status 10))
-  (segment (start 84.19 59.5) (end 81 59.5) (width 0.25) (layer F.Cu) (net 8))
-  (segment (start 78.5 57) (end 78.5 48.225) (width 0.25) (layer F.Cu) (net 8))
-  (segment (start 81 59.5) (end 78.5 57) (width 0.25) (layer F.Cu) (net 8))
+  (segment (start 84.19 59.5) (end 83.25 59.5) (width 0.25) (layer F.Cu) (net 8))
+  (segment (start 78.5 54.75) (end 78.5 48.225) (width 0.25) (layer F.Cu) (net 8))
+  (segment (start 83.25 59.5) (end 78.5 54.75) (width 0.25) (layer F.Cu) (net 8))
   (segment (start 84.19 59.5) (end 84.19 59.44) (width 0.25) (layer F.Cu) (net 8))
   (segment (start 77 48.225) (end 78.5 48.225) (width 0.25) (layer F.Cu) (net 8))
@@
   (segment (start 122.25 59.5) (end 123.75 61) (width 0.25) (layer F.Cu) (net 8))
   (segment (start 139.69 61) (end 141.19 59.5) (width 0.25) (layer F.Cu) (net 8))
-  (segment (start 123.75 61) (end 139.69 61) (width 0.25) (layer F.Cu) (net 8))
+  (segment (start 123.75 61) (end 132.5 61) (width 0.25) (layer F.Cu) (net 8))
+  (segment (start 132.5 61) (end 134 62.5) (width 0.25) (layer F.Cu) (net 8))
+  (segment (start 134 62.5) (end 137 62.5) (width 0.25) (layer F.Cu) (net 8))
+  (segment (start 137 62.5) (end 138.5 61) (width 0.25) (layer F.Cu) (net 8))
+  (segment (start 138.5 61) (end 139.69 61) (width 0.25) (layer F.Cu) (net 8))
   (segment (start 141.19 59.5) (end 141.25 59.5) (width 0.25) (layer F.Cu) (net 8))
   (segment (start 42 48.225) (end 42 46.19) (width 0.25) (layer B.Cu) (net 8))
@@
   (segment (start 123 61) (end 114.25 61) (width 0.25) (layer F.Cu) (net 16))
   (segment (start 123.5 61.5) (end 123 61) (width 0.25) (layer F.Cu) (net 16))
-  (segment (start 133 61.5) (end 123.5 61.5) (width 0.25) (layer F.Cu) (net 16))
+  (segment (start 131.5 61.5) (end 123.5 61.5) (width 0.25) (layer F.Cu) (net 16))
   (segment (start 172 65.19) (end 171.94 65.19) (width 0.25) (layer F.Cu) (net 16))
   (segment (start 171.94 65.19) (end 169.25 62.5) (width 0.25) (layer F.Cu) (net 16))
@@
   (segment (start 80.06 65.19) (end 82.75 62.5) (width 0.25) (layer F.Cu) (net 16))
   (segment (start 82.75 62.5) (end 93.99 62.5) (width 0.25) (layer F.Cu) (net 16))
-  (segment (start 134 65.19) (end 134 62.5) (width 0.25) (layer F.Cu) (net 16))
-  (segment (start 134 62.5) (end 133 61.5) (width 0.25) (layer F.Cu) (net 16))
-  (segment (start 84.19 78.5) (end 81 78.5) (width 0.25) (layer F.Cu) (net 16))
-  (segment (start 78.5 76) (end 78.5 65.19) (width 0.25) (layer F.Cu) (net 16))
-  (segment (start 81 78.5) (end 78.5 76) (width 0.25) (layer F.Cu) (net 16))
+  (segment (start 134 65.19) (end 134 64) (width 0.25) (layer F.Cu) (net 16))
+  (segment (start 134 64) (end 131.5 61.5) (width 0.25) (layer F.Cu) (net 16))
+  (segment (start 84.19 78.5) (end 83.25 78.5) (width 0.25) (layer F.Cu) (net 16))
+  (segment (start 78.5 73.75) (end 78.5 65.19) (width 0.25) (layer F.Cu) (net 16))
+  (segment (start 83.25 78.5) (end 78.5 73.75) (width 0.25) (layer F.Cu) (net 16))
   (segment (start 137 65.19) (end 137.06 65.19) (width 0.25) (layer F.Cu) (net 16))
   (segment (start 134 65.19) (end 137 65.19) (width 0.25) (layer F.Cu) (net 16))
@@
   (segment (start 160.19 90.73) (end 160.19 90.54) (width 0.25) (layer F.Cu) (net 31))
   (segment (start 172 91.81) (end 172 89.775) (width 0.25) (layer B.Cu) (net 31))
+  (segment (start 137 103.19) (end 137 105.225) (width 0.25) (layer F.Cu) (net 32) (status C00000))
+  (segment (start 134 103.19) (end 134 105.225) (width 0.25) (layer F.Cu) (net 32) (status C00000))
   (segment (start 99 103.19) (end 99 105.225) (width 0.25) (layer B.Cu) (net 32))
   (segment (start 137 103.19) (end 137.06 103.19) (width 0.25) (layer F.Cu) (net 32))
@@
   (segment (start 172 103.19) (end 172 105.225) (width 0.25) (layer B.Cu) (net 32))
   (segment (start 172 103.19) (end 172 105.225) (width 0.25) (layer F.Cu) (net 32))
-  (segment (start 134 103.19) (end 134 105.225) (width 0.25) (layer F.Cu) (net 32))
   (segment (start 134 105.225) (end 134 106.5) (width 0.25) (layer F.Cu) (net 32))
   (segment (start 134 106.5) (end 134.25 106.75) (width 0.25) (layer F.Cu) (net 32))
@@
   (segment (start 134.3 48.8) (end 136.75 48.8) (width 0.25) (layer B.Cu) (net 49))
   (segment (start 124 37.5) (end 124.25 37.75) (width 0.25) (layer F.Cu) (net 50))
-  (segment (start 124 37.5) (end 101.25 37.5) (width 0.25) (layer F.Cu) (net 50))
+  (segment (start 124 37.5) (end 122.25 37.5) (width 0.25) (layer F.Cu) (net 50))
+  (segment (start 122.25 37.5) (end 121.375 39.25) (width 0.25) (layer F.Cu) (net 50))
+  (segment (start 121.375 39.25) (end 119.625 39.25) (width 0.25) (layer F.Cu) (net 50))
+  (segment (start 119.625 39.25) (end 118.75 37.5) (width 0.25) (layer F.Cu) (net 50))
+  (segment (start 118.75 37.5) (end 101.25 37.5) (width 0.25) (layer F.Cu) (net 50))
   (segment (start 101.25 37.5) (end 100.75 38) (width 0.25) (layer F.Cu) (net 50))
   (segment (start 100.75 38) (end 100.75 40.5) (width 0.25) (layer F.Cu) (net 50))

Commit message: Fix lines and add text of author
Parts:
- RESET: renamed from RSW1; moved to B.Cu
- moved RESET 5.00 mm to (123.0, 39.2), turned to 180 degrees
- renumbered C2 to GND, C3 to LED, J1 to TRS, C1 to VCC
Routing:
- net col0: track 264.7 -> 296.9 mm
- net col6: track 217.0 -> 248.7 mm
- net row4: track 276.4 -> 300.0 mm, vias 8 -> 6
- net row3: track 256.8 -> 276.1 mm
- net reset: track 8.13 -> 12.8 mm
Other:
- board size 132 x 98 mm -> 132 x 98.5 mm
- board text added: "Waffle PCB v0.1 PCB Designed by foostan"

Commit message: Add waffle logo
Parts:
- added G***: LOGO, kbd:waffle, F.Cu at (98.2, 78.8)
- added G***: LOGO, kbd:waffle, B.Cu at (127.5, 80.0)
